File: electrical/eis.kicad_sch (KiCad schematic)
At the start: 53 parts

Commit message: Upgraded G3X Touch to Axis
Parts:
- CARB_TEMP, CAUTION, CHT1P, CHT1R, CHT2P, CHT2R, CHT3P, CHT3R, CHT4P, CHT4R, EGT1P, EGT1R, EGT2P, EGT2R, EGT3P, EGT3R, EGT4P, EGT4R, FLAPS_POS, FUEL_LEFT, FUEL_RIGHT, GEA24, OIL_TEMP, SureFly_TACH1, WARNING: value ~ -> (none)
