File: electrical/lights.kicad_sch (KiCad schematic)
At the start: 22 parts

Commit message: Upgraded G3X Touch to Axis
Parts:
- FL_CONTROLLER, FL_TAIL1, FL_TIP_LT, FL_TIP_RT, LANDING_TIP_LT, LANDING_TIP_RT, LANDING_WING_LT, LANDING_WING_RT, POSITION_SW1, STROBE_SW1, TAXI_SW1, TAXI_WING_LT: value ~ -> (none)
