File: electrical/lycoming.kicad_sch (KiCad schematic)
At the start: 26 parts

Commit message: Upgraded G3X Touch to Axis
Parts:
- added GDU_BAT_F: 2A, symbol Device:Fuse
- added GDU_BAT_SW: (no value), symbol Switch:SW_SPST
- ALT_SW, BAK_SW, MAG_LEFT_SW, MAG_RIGHT_SW, MAIN_SW, SFLY_LEFT, SFLY_RIGHT: value ~ -> (none)
Connections:
- net BAK_BATTERY_VOLTS: now also GDU_BAT_F.2
- new net: GDU_BAT_F.1, GDU_BAT_SW.1 (A)
- new net GDU_BAT: GDU_BAT_SW.2 (B)
