File: electrical/power.kicad_sch (KiCad schematic)
At the start: 48 parts

Commit message: Upgraded G3X Touch to Axis
Parts:
- 12V_SW, AVIONICS_SW, FUEL_PUMP_SW, IGN_BAK, IGN_BAK_SW, SMOKE_SW: value ~ -> (none)
